File: Calavera.kicad_pcb (KiCad board)
At the start: 2 copper layers, 39.2 x 59.2 mm, 24 parts, among them Q1 Q_DUAL_NMOS, U1 AT42QT1012, U2 LMV932

Commit message: 4 Layer test
Routing:
- added copper zone on In1.Cu, net GND
Other:
- copper layers 2 -> 4
Changed lines of the file:
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@@
   (layers
     (0 F.Cu signal hide)
+    (1 In1.Cu signal)
+    (2 In2.Cu signal)
     (31 B.Cu signal)
     (32 B.Adhes user)
-    (33 F.Adhes user hide)
-    (34 B.Paste user hide)
-    (35 F.Paste user hide)
+    (33 F.Adhes user)
+    (34 B.Paste user)
+    (35 F.Paste user)
     (36 B.SilkS user)
     (37 F.SilkS user hide)
-    (38 B.Mask user hide)
+    (38 B.Mask user)
     (39 F.Mask user hide)
     (40 Dwgs.User user)
@@
     (44 Edge.Cuts user)
     (45 Margin user)
-    (46 B.CrtYd user hide)
-    (47 F.CrtYd user hide)
+    (46 B.CrtYd user)
+    (47 F.CrtYd user)
     (48 B.Fab user)
-    (49 F.Fab user hide)
+    (49 F.Fab user)
   )
   (setup
@@
       )
     )
+  )
+  (zone (net 3) (net_name GND) (layer In1.Cu) (hatch edge 0.508)
+    (connect_pads (clearance 0))
+    (min_thickness 0.254)
+    (fill yes (arc_segments 32) (thermal_gap 0.508) (thermal_bridge_width 0.508))
+    (polygon
+      (pts
+        (xy 135.55 117.45) (xy 142.1 117.4) (xy 143.2 121.7) (xy 139.65 126.55) (xy 133.65 121.15)
+        (xy 135.5 117.45)
+      )
+    )

Commit message: added layer in2
Routing:
- added copper zone on In2.Cu, net GND
Changed lines of the file:
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@@
+    )
+  )
+  (zone (net 3) (net_name GND) (layer In2.Cu) (hatch edge 0.508)
+    (connect_pads (clearance 0))
+    (min_thickness 0.254)
+    (fill yes (arc_segments 32) (thermal_gap 0.508) (thermal_bridge_width 0.508))
+    (polygon
+      (pts
+        (xy 128.65 106.45) (xy 137.65 118.5) (xy 136.1 122.1) (xy 130.65 117.1) (xy 126.75 108.1)
+      )
     )
   )

Commit message: no message
Routing:
- net GND: track 0.00 -> 13.5 mm
Changed lines of the file:
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@@
     (thickness 1.6)
     (drawings 3)
-    (tracks 150)
+    (tracks 154)
     (zones 0)
     (modules 24)
@@
     (1 In1.Cu signal)
     (2 In2.Cu signal)
-    (31 B.Cu signal)
+    (31 B.Cu signal hide)
     (32 B.Adhes user)
     (33 F.Adhes user)
@@
   (via (at 143.3 80.1) (size 0.6) (drill 0.4) (layers F.Cu B.Cu) (net 3))
   (via (at 139.2 74.84) (size 2.01) (drill 2) (layers F.Cu B.Cu) (net 3))
+  (segment (start 136.6 95.6) (end 139.85 95.6) (width 0.25) (layer In2.Cu) (net 3))
+  (segment (start 139.85 95.6) (end 141.7 95.6) (width 0.25) (layer In2.Cu) (net 3))
+  (segment (start 135.324264 80.1) (end 143.3 80.1) (width 0.25) (layer In1.Cu) (net 3))
+  (segment (start 134.9 80.1) (end 135.324264 80.1) (width 0.25) (layer In1.Cu) (net 3))
   (segment (start 142.965 97.14) (end 143 97.175) (width 0.25) (layer B.Cu) (net 4) (status 30))
   (segment (start 140.63 97.14) (end 142.965 97.14) (width 0.25) (layer B.Cu) (net 4) (status 30))
