File: Calavera.sch (KiCad schematic (older format))
At the start: 24 parts, among them Q1 Q_DUAL_NMOS, U1 AT42QT1012, U2 LMV932

Commit message: Put everything on a single library, and the 3D models are now relative to the project path
Parts:
- C1, C2, C3: footprint felcana:0805-C_Handsolder -> Calavera:0805-C_Handsolder
- R1, R10, R2, R3, R4, R5, R6, R7, R8, R9: footprint felcana:0805-R_Handsolder -> Calavera:0805-R_Handsolder
Changed lines of the file:
@@
 F 0 "R1" V 1545 1800 50  0000 C CNN
 F 1 "10kΩ" V 1636 1800 50  0000 C CNN
-F 2 "felcana:0805-R_Handsolder" H 1750 1800 50  0001 C CNN
+F 2 "Calavera:0805-R_Handsolder" H 1750 1800 50  0001 C CNN
 F 3 "~" H 1750 1800 50  0001 C CNN
 	1    1750 1800
@@
 F 0 "C1" H 2042 2046 50  0000 L CNN
 F 1 "22nF" H 2042 1955 50  0000 L CNN
-F 2 "felcana:0805-C_Handsolder" H 1950 2000 50  0001 C CNN
+F 2 "Calavera:0805-C_Handsolder" H 1950 2000 50  0001 C CNN
 F 3 "~" H 1950 2000 50  0001 C CNN
 	1    1950 2000
@@
 F 0 "R2" H 2018 2346 50  0000 L CNN
 F 1 "1MΩ" H 2018 2255 50  0000 L CNN
-F 2 "felcana:0805-R_Handsolder" H 1950 2300 50  0001 C CNN
+F 2 "Calavera:0805-R_Handsolder" H 1950 2300 50  0001 C CNN
 F 3 "~" H 1950 2300 50  0001 C CNN
 	1    1950 2300
@@
 F 0 "R3" H 3468 2046 50  0000 L CNN
 F 1 "100kΩ" H 3468 1955 50  0000 L CNN
-F 2 "felcana:0805-R_Handsolder" H 3400 2000 50  0001 C CNN
+F 2 "Calavera:0805-R_Handsolder" H 3400 2000 50  0001 C CNN
 F 3 "~" H 3400 2000 50  0001 C CNN
 	1    3400 2000
@@
 F 0 "C2" H 2442 1446 50  0000 L CNN
 F 1 "100nF" H 2442 1355 50  0000 L CNN
-F 2 "felcana:0805-C_Handsolder" H 2350 1400 50  0001 C CNN
+F 2 "Calavera:0805-C_Handsolder" H 2350 1400 50  0001 C CNN
 F 3 "~" H 2350 1400 50  0001 C CNN
 	1    2350 1400
@@
 F 0 "R4" H 6168 3746 50  0000 L CNN
 F 1 "R_Small_US" H 6168 3655 50  0000 L CNN
-F 2 "felcana:0805-R_Handsolder" H 6100 3700 50  0001 C CNN
+F 2 "Calavera:0805-R_Handsolder" H 6100 3700 50  0001 C CNN
 F 3 "~" H 6100 3700 50  0001 C CNN
 	1    6100 3700
@@
 F 0 "R5" H 6818 3746 50  0000 L CNN
 F 1 "R_Small_US" H 6818 3655 50  0000 L CNN
-F 2 "felcana:0805-R_Handsolder" H 6750 3700 50  0001 C CNN
+F 2 "Calavera:0805-R_Handsolder" H 6750 3700 50  0001 C CNN
 F 3 "~" H 6750 3700 50  0001 C CNN
 	1    6750 3700
@@
 F 0 "C3" H 7092 1296 50  0000 L CNN
 F 1 "22μF" H 7092 1205 50  0000 L CNN
-F 2 "felcana:0805-C_Handsolder" H 7000 1250 50  0001 C CNN
+F 2 "Calavera:0805-C_Handsolder" H 7000 1250 50  0001 C CNN
 F 3 "~" H 7000 1250 50  0001 C CNN
 	1    7000 1250
@@
 F 0 "R7" H 7668 1846 50  0000 L CNN
 F 1 "1200Ω" H 7668 1755 50  0000 L CNN
-F 2 "felcana:0805-R_Handsolder" H 7600 1800 50  0001 C CNN
+F 2 "Calavera:0805-R_Handsolder" H 7600 1800 50  0001 C CNN
 F 3 "~" H 7600 1800 50  0001 C CNN
 	1    7600 1800
@@
 F 0 "R8" H 8318 1446 50  0000 L CNN
 F 1 "8200Ω" H 8318 1355 50  0000 L CNN
-F 2 "felcana:0805-R_Handsolder" H 8250 1400 50  0001 C CNN
+F 2 "Calavera:0805-R_Handsolder" H 8250 1400 50  0001 C CNN
 F 3 "~" H 8250 1400 50  0001 C CNN
 	1    8250 1400
@@
 F 0 "R6" H 6118 1946 50  0000 L CNN
 F 1 "180kΩ" H 6118 1855 50  0000 L CNN
-F 2 "felcana:0805-R_Handsolder" H 6050 1900 50  0001 C CNN
+F 2 "Calavera:0805-R_Handsolder" H 6050 1900 50  0001 C CNN
 F 3 "~" H 6050 1900 50  0001 C CNN
 	1    6050 1900
@@
 F 0 "R9" H 9768 1646 50  0000 L CNN
 F 1 "2490" H 9768 1555 50  0000 L CNN
-F 2 "felcana:0805-R_Handsolder" H 9700 1600 50  0001 C CNN
+F 2 "Calavera:0805-R_Handsolder" H 9700 1600 50  0001 C CNN
 F 3 "~" H 9700 1600 50  0001 C CNN
 	1    9700 1600
@@
 F 0 "R10" H 9768 1946 50  0000 L CNN
 F 1 "10kΩ" H 9768 1855 50  0000 L CNN
-F 2 "felcana:0805-R_Handsolder" H 9700 1900 50  0001 C CNN
+F 2 "Calavera:0805-R_Handsolder" H 9700 1900 50  0001 C CNN
 F 3 "~" H 9700 1900 50  0001 C CNN
 	1    9700 1900
