File: hardware/Calavera.sch (KiCad schematic (older format))
At the start: 24 parts, among them Q1 Q_DUAL_NMOS, U1 AT42QT1012, U2 LMV932

Commit message: Cleaning here and there
Parts:
- Q1: MPN NX138BKS -> DMN2004DMK
Changed lines of the file:
@@
 F 1 "Q_DUAL_NMOS" H 4050 3800 50  0001 L CNN
 F 2 "Calavera:SOT23-6-NMOSx2_Handsolder" H 4600 3750 50  0001 C CNN
-F 3 "https://assets.nexperia.com/documents/data-sheet/NX138BKS.pdf" H 4050 3900 50  0001 C CNN
+F 3 "https://www.diodes.com/assets/Datasheets/ds30937.pdf" H 4050 3900 50  0001 C CNN
 	2    3850 3900
 	-1   0    0    -1
@@
 F 1 "Q_DUAL_NMOS" H 3200 3900 50  0001 L CNN
 F 2 "Calavera:SOT23-6-NMOSx2_Handsolder" H 3750 3750 50  0001 C CNN
-F 3 "https://assets.nexperia.com/documents/data-sheet/NX138BKS.pdf" H 3200 3900 50  0001 C CNN
-F 4 "NX138BKS" H 3000 3900 50  0001 C CNN "MPN"
+F 3 "https://www.diodes.com/assets/Datasheets/ds30937.pdf" H 3200 3900 50  0001 C CNN
+F 4 "DMN2004DMK" H 3000 3900 50  0001 C CNN "MPN"
 	1    3000 3900
 	1    0    0    -1
