File: hardware/Calavera.kicad_sch (KiCad schematic)
At the start: 24 parts, among them Q1 DMN65D8L, SW1 SW_SPDT, U1 AT42QT1012, U2 LMV932

Commit message: 3D model behaves again
Parts:
- D1, D2, R6, R7: Digikey PN (none) -> N/A; Farnell PN (none) -> N/A; MPN (none) -> N/A; Manufacturer  (none) -> N/A
- R1, R11, R9: Digikey PN 311-10KARCT-ND -> CR0805-FX-1002ELFCT-ND; Farnell PN 2073612 -> 1612522; MPN RC0805JR-0710KL -> CR0805-FX-1002ELF; Manufacturer  Yageo -> Bourns Inc.; Tolerance (none) -> ±1%, 1/8W; VRating (none) -> 150V
- R10: Digikey PN (none) -> CR0805-FX-2491ELFCT-ND; Farnell PN (none) -> 3540417; MPN (none) -> CR0805-FX-2491ELF; Manufacturer  (none) -> Bourns Inc.; Tolerance (none) -> ±1%, 1/8W; VRating (none) -> 150V
- R2: Digikey PN (none) -> CR0805-FX-1004ELFCT-ND; Farnell PN (none) -> 2333538; MPN (none) -> CR0805-FX-1004ELF; Manufacturer  (none) -> Bourns Inc.; Tolerance (none) -> ±1%, 1/8W; VRating (none) -> 150V
- R3, R4, R5: Digikey PN (none) -> CR0805-FX-1003ELFCT-ND; Farnell PN (none) -> 2333577; MPN (none) -> CR0805-FX-1003ELF; Manufacturer  (none) -> Bourns Inc.; Tolerance (none) -> ±1%, 1/8W; VRating (none) -> 150V
- R8: value 1470Ω -> 1k5Ω; Digikey PN (none) -> CR0805-FX-1501ELFCT-ND; Farnell PN (none) -> 2333560; MPN (none) -> CR0805-FX-1501ELF; Manufacturer  (none) -> Bourns Inc.; Tolerance (none) -> ±1%, 1/8W; VRating (none) -> 150V
